Commit message: [add] livox mesh and factory world

File: sjtu_drone_description/urdf/drone.urdf (robot description, URDF)
Before this commit: robot sjtu_drone, 5 links, 4 joints
Links:
- added link upper_lidar_link
Joints:
- added joint upper_lidar_joint: type fixed, parent base_link, child upper_lidar_link, origin xyz=0 0 0.5 rpy=0 0 0
