Commit message: [mod] correct xacro file with lidar

File: sjtu_drone_description/urdf/sjtu_drone_lidar.urdf.xacro (robot description, xacro)
@@ -24,6 +24,5 @@
       <origin rpy="0 0 0" xyz="0   0   0.04"/>
       <geometry>
-        <mesh filename="file:/home/ws/src/sjtu_drone/sjtu_drone_description/models/sjtu_drone/quadrotor_4.stl"/>
-        <!-- <mesh filename="file://$(find sjtu_drone_description)/models/sjtu_drone/quadrotor_4.stl"/> -->
+        <mesh filename="file://$(find sjtu_drone_description)/models/sjtu_drone/quadrotor_4.stl"/>
         <!-- <mesh filename="package://sjtu_drone/quadrotor_4.stl"/> -->
       </geometry>
@@ -32,6 +31,5 @@
       <origin rpy="0 0 0" xyz="0   0   0.04"/>
       <geometry>
-        <mesh filename="file:/home/ws/src/sjtu_drone/sjtu_drone_description/models/sjtu_drone/quadrotor_4.dae"/>
-        <!-- <mesh filename="file://$(find sjtu_drone_description)/models/sjtu_drone/quadrotor_4.dae"/> -->
+        <mesh filename="file://$(find sjtu_drone_description)/models/sjtu_drone/quadrotor_4.dae"/>
         <!-- <mesh filename="package://sjtu_drone/quadrotor_4.dae"/> -->
       </geometry>
@@ -54,6 +52,6 @@
       <origin rpy="1.6 0 0" xyz="0   0   0.14"/>
       <geometry>
-        <mesh filename="file:/home/ws/src/sjtu_drone/sjtu_drone_description/models/mid-360-asm.dae" scale="0.002 0.002 0.002"/>
-        <!-- <mesh filename="file://$(find sjtu_drone_description)/models/mid-360-asm.dae" scale="0.002 0.002 0.002"/> -->
+        <!-- <mesh filename="file:/home/ws/src/sjtu_drone/sjtu_drone_description/models/mid-360-asm.dae" scale="0.002 0.002 0.002"/> -->
+        <mesh filename="file://$(find sjtu_drone_description)/models/mid-360-asm.dae" scale="0.002 0.002 0.002"/>
         <!--/home/mea/dev_ws/src/sjtu_drone/sjtu_drone_description/models/mid-360-asm.dae-->
         <!-- <mesh filename="package://sjtu_drone/quadrotor_4.stl"/> -->
@@ -121,5 +119,5 @@
       <always_on> 1 </always_on>
       <visualize>1</visualize>
-      <update_rate> 5 </update_rate>
+      <update_rate> 100 </update_rate>
       <pose> 0 0 0 0 0 0 </pose>
       <imu>
@@ -151,5 +149,5 @@
       <always_on>1</always_on>
       <visualize>1</visualize>
-      <update_rate>1</update_rate>
+      <update_rate>30</update_rate>
       <ray>
         <scan>
@@ -228,5 +226,5 @@
         <frame_name>${mp['namespace']}/lidar_link</frame_name>
         <organize_cloud>false</organize_cloud>
-        <!--output_type>sensor_msgs/Range</output_type-->
+        <!-- <output_type>sensor_msgs/Range</output_type> -->
         <radiation_type>ultrasound</radiation_type>
         <min_range>0.3</min_range>
@@ -239,5 +237,5 @@
       <always_on>1</always_on>
       <visualize>1</visualize>
-      <update_rate>5</update_rate>
+      <update_rate>60</update_rate>
       <camera>
         <horizontal_fov>2.09</horizontal_fov>
@@ -274,5 +272,5 @@
       <always_on>1</always_on>
       <visualize>1</visualize>
-      <update_rate>5</update_rate>
+      <update_rate>15</update_rate>
       <camera>
         <horizontal_fov>1.047</horizontal_fov>
@@ -307,5 +305,5 @@
     <sensor name="gps" type="gps">
       <always_on>1</always_on>
-      <update_rate>5</update_rate>
+      <update_rate>30</update_rate>
       <gps>
         <position_sensing>
@@ -335,5 +333,5 @@
   <gazebo reference="base_link">
     <sensor name="collision_sensor" type="contact">
-      <update_rate>5.0</update_rate>
+      <update_rate>100</update_rate>
       <always_on>true</always_on>
       <contact>
